File: long.sch (EAGLE design)
At the start: 20 parts, among them U1 USD-SOCKET, U2 MCP73831, U3 TPS61200, X1 Micro USB

Commit message: Added round boards
Parts:
- added JP1, JP2, JP3, JP4, JP5, JP6, JP8, JP9: (no value), pinhead:PINHD-1X4
- added U$2: UBLOX_MAX, Ava:UBLOX_MAX
- added U$3: ADXL377, SparkFun-Sensors:ADXL377
Changed lines of the file:
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@@
 <?xml version="1.0" encoding="utf-8"?>
 <!DOCTYPE eagle SYSTEM "eagle.dtd">
-<eagle version="7.2.0">
+<eagle version="7.0.0">
 <drawing>
 <settings>
@@
 <part name="C6" library="CH_passive" deviceset="CAP" device="1206" value="10uF"/>
 <part name="L1" library="SparkFun" deviceset="INDUCTOR" device="." value="4.7uH, 1.2A"/>
+<part name="U$2" library="Ava" deviceset="UBLOX_MAX" device=""/>
+<part name="JP1" library="pinhead" deviceset="PINHD-1X4" device=""/>
+<part name="JP2" library="pinhead" deviceset="PINHD-1X4" device=""/>
+<part name="JP3" library="pinhead" deviceset="PINHD-1X4" device=""/>
+<part name="JP4" library="pinhead" deviceset="PINHD-1X4" device=""/>
+<part name="JP5" library="pinhead" deviceset="PINHD-1X4" device=""/>
+<part name="JP6" library="pinhead" deviceset="PINHD-1X4" device=""/>
+<part name="JP8" library="pinhead" deviceset="PINHD-1X4" device=""/>
+<part name="JP9" library="pinhead" deviceset="PINHD-1X4" device=""/>
+<part name="U$3" library="SparkFun-Sensors" deviceset="ADXL377" device=""/>
 </parts>
 <sheets>
@@
 <attribute name="VALUE" x="210.82" y="45.72" size="1.778" layer="96"/>
 </instance>
+<instance part="U$2" gate="G$1" x="187.96" y="119.38"/>
+<instance part="JP1" gate="A" x="238.76" y="124.46"/>
+<instance part="JP2" gate="A" x="251.46" y="124.46"/>
+<instance part="JP3" gate="A" x="264.16" y="124.46"/>
+<instance part="JP4" gate="A" x="276.86" y="124.46"/>
+<instance part="JP5" gate="A" x="238.76" y="104.14"/>
+<instance part="JP6" gate="A" x="251.46" y="104.14"/>
+<instance part="JP8" gate="A" x="264.16" y="104.14"/>
+<instance part="JP9" gate="A" x="276.86" y="104.14"/>
+<instance part="U$3" gate="G$1" x="238.76" y="71.12"/>
 </instances>
 <busses>

Commit message: Added ADXL375 library
Parts:
- removed U$3: ADXL377, SparkFun-Sensors:ADXL377
- added U4: ADXL375BCCZ, adxl375bccz:ADXL375BCCZ
Changed lines of the file:
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@@
 <part name="JP8" library="pinhead" deviceset="PINHD-1X4" device=""/>
 <part name="JP9" library="pinhead" deviceset="PINHD-1X4" device=""/>
-<part name="U$3" library="SparkFun-Sensors" deviceset="ADXL377" device=""/>
+<part name="U4" library="adxl375bccz" deviceset="ADXL375BCCZ" device=""/>
 </parts>
 <sheets>
@@
 <instance part="JP8" gate="A" x="264.16" y="104.14"/>
 <instance part="JP9" gate="A" x="276.86" y="104.14"/>
-<instance part="U$3" gate="G$1" x="238.76" y="71.12"/>
+<instance part="U4" gate="A" x="322.58" y="119.38"/>
 </instances>
 <busses>
