File: sensorBoard.sch (EAGLE design)
At the start: 0 parts

Commit message: Created schematic
Parts:
- added C1, C2, C3, C6: 100n, rcl:C-EUC0402
- added C4: 10n, rcl:C-EUC0402
- added C5: 4.7uF, rcl:C-EUC0402
- added C7: 220n, rcl:C-EUC0402
- added JP1, JP2: (no value), SparkFun:M03PTH
- added JP3, JP4: (no value), SparkFun:M05PTH
- added Q1: BSS84, transistor-small-signal:BSS84
- added U$1: UBLOX_MAX, Ava:UBLOX_MAX
- added U$2: HMC5883LSMD, SparkFun:HMC5883LSMD
- added U$3: KSSG74B16, mattsLib:KSSG74B16
- added U$4: PCAL9554B, mattsLib:PCAL9554B
- added U$5, U$6, U$7, U$8: SIA448DJ, mattsLib:SIA448DJ
- added U1: ADXL345, SparkFun:ADXL345
- added U2: L3G4200D, SparkFun:L3G4200D
- added U3: MPL115A, SparkFun:MPL115A
- added X2, X3: (no value), con-molex:22-23-2061
Connections:
- new net EXT_CS: JP4.3
- new net EXT_MISO: JP4.4
- new net EXT_MOSI: JP4.2
- new net EXT_RX: JP2.2
- new net EXT_SCK: JP4.5
- new net EXT_TX: JP2.3
- new net GND: C1.2, C2.2, C3.2, C4.2, C5.2, JP1.3, Q1.D, U$1.10_GND, U$1.12_GND, U$1.1_GND, U$2.GND@1, U$2.GND@2, U$4.A0, U$4.A1, U$4.A2, U$4.VSS, U$5.S, U$6.S, U$7.S, U$8.S, U1.GND@2, U1.GND@4, U1.GND@5, U2.GND, U2.RSDVG@3, U2.RSVDG@1, U2.RSVDG@2, U2.RSVDG@4, U3.GND, X2-6.S, X3-6.S
- new net GPIO1: JP3.1, Q1.G
- new net GPIO2: JP3.2
- new net GPIO3: JP3.3
- new net GPS_RX: JP4.1, U$1.3_RXD1
- new net GPS_TX: JP3.5, U$1.2_TXD1
- new net HP0: U$5.D, X2-2.S
- new net HP1: U$6.D, X2-3.S
- new net HP2: U$7.D, X2-4.S
- new net HP3: U$8.D, X2-5.S
- new net I2C_SCL: JP1.1, U$2.SCL, U$4.SCL, U1.SCL, U2.SCL, U3.SCLK
- new net I2C_SDA: JP2.1, U$2.SDA, U$4.SDA, U1.SDA, U2.SDA/SDI, U3.SDA/DIN
- new net N$1: C4.1, U2.PLL
- new net N$2: C5.1, C6.2, U$2.C1
- new net N$3: C7.2, U$2.SETC
- new net N$4: C7.1, U$2.SETP
- new net N$5: Q1.S, U$3.-
- new net P0: U$4.P0, U$5.G
- new net P1: U$4.P1, U$6.G
- new net P2: U$4.P2, U$7.G
- new net P3: U$4.P3, U$8.G
- new net P4: U$4.P4, X3-2.S
- new net P5: U$4.P5, X3-3.S
- new net P6: U$4.P6, X3-4.S
- new net P7: U$4.P7, X3-5.S
- new net VBAT: JP3.4, U$3.+
- new net VCC: C1.1, C2.1, C3.1, C6.1, JP1.2, U$1.6_V_BCKP, U$1.7_VCC_IO, U$1.8_VCC, U$1.9_V_RESET, U$2.S1, U$2.VDD, U$2.VDDIO, U$4.VDD, U1.VDD, U1.VSS, U2.RSVDV@0, U2.VDD, U2.VDDIO, U3.SHDN, U3.VDD
- new net V_BAT: X2-1.S, X3-1.S
