File: sensorBoard.sch (EAGLE design)
At the start: 25 parts, among them Q1 BSS84, U1 ADXL345, U2 L3G4200D, U3 MPL115A

Commit message: Changed schematic, positioned components
Parts:
- removed X2, X3: (no value), con-molex:22-23-2061
- added JP5: (no value), SparkFun:M06SIP
- added U$9: JTI_ANTENNA-1575AT43A40, Ava:JTI_ANTENNA-1575AT43A40
- added X1: 22-23-2051, con-molex:22-23-2051
Connections:
- removed net V_BAT: X2-1.S, X3-1.S
- new net N$6: U$1.11_RF_IN, U$9.FEED
- net GND: now also X1-5.S; no longer X2-6.S, X3-6.S
- net GPIO1: now also JP5.5; no longer Q1.G
- net GPIO2: now also JP5.6
- net GPIO3: now also Q1.G
- net HP0: now also X1-1.S; no longer X2-2.S
- net HP1: now also X1-2.S; no longer X2-3.S
- net HP2: now also X1-3.S; no longer X2-4.S
- net HP3: now also X1-4.S; no longer X2-5.S
- net P4: now also JP5.1; no longer X3-2.S
- net P5: now also JP5.2; no longer X3-3.S
- net P6: now also JP5.3; no longer X3-4.S
- net P7: now also JP5.4; no longer X3-5.S
Changed lines of the file:
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@@
 <part name="U$7" library="mattsLib" deviceset="SIA448DJ" device=""/>
 <part name="U$8" library="mattsLib" deviceset="SIA448DJ" device=""/>
-<part name="X2" library="con-molex" deviceset="22-23-2061" device=""/>
-<part name="X3" library="con-molex" deviceset="22-23-2061" device=""/>
 <part name="GND10" library="supply1" deviceset="GND" device=""/>
-<part name="GND11" library="supply1" deviceset="GND" device=""/>
 <part name="GND12" library="supply1" deviceset="GND" device=""/>
+<part name="X1" library="con-molex" deviceset="22-23-2051" device=""/>
+<part name="JP5" library="SparkFun" deviceset="M06" device="SIP"/>
+<part name="U$9" library="Ava" deviceset="JTI_ANTENNA-1575AT43A40" device=""/>
 </parts>
 <sheets>
@@
 <instance part="U$7" gate="G$1" x="248.92" y="45.72"/>
 <instance part="U$8" gate="G$1" x="261.62" y="45.72"/>
-<instance part="X2" gate="-1" x="231.14" y="27.94"/>
-<instance part="X2" gate="-2" x="231.14" y="25.4"/>
-<instance part="X2" gate="-3" x="231.14" y="22.86"/>
-<instance part="X2" gate="-4" x="231.14" y="20.32"/>
-<instance part="X2" gate="-5" x="231.14" y="17.78"/>
-<instance part="X2" gate="-6" x="231.14" y="15.24"/>
-<instance part="X3" gate="-1" x="256.54" y="27.94"/>
-<instance part="X3" gate="-2" x="256.54" y="25.4"/>
-<instance part="X3" gate="-3" x="256.54" y="22.86"/>
-<instance part="X3" gate="-4" x="256.54" y="20.32"/>
-<instance part="X3" gate="-5" x="256.54" y="17.78"/>
-<instance part="X3" gate="-6" x="256.54" y="15.24"/>
 <instance part="GND10" gate="1" x="223.52" y="12.7"/>
-<instance part="GND11" gate="1" x="248.92" y="12.7"/>
 <instance part="GND12" gate="1" x="241.3" y="33.02"/>
+<instance part="X1" gate="-1" x="231.14" y="25.4"/>
+<instance part="X1" gate="-2" x="231.14" y="22.86"/>
+<instance part="X1" gate="-3" x="231.14" y="20.32"/>
+<instance part="X1" gate="-4" x="231.14" y="17.78"/>
+<instance part="X1" gate="-5" x="231.14" y="15.24"/>
+<instance part="JP5" gate="G$1" x="259.08" y="20.32" rot="R180"/>
+<instance part="U$9" gate="G$1" x="12.7" y="99.06" rot="R180"/>
 </instances>
 <busses>
@@
 </segment>
 <segment>
-<pinref part="X2" gate="-6" pin="S"/>
 <wire x1="228.6" y1="15.24" x2="223.52" y2="15.24" width="0.1524" layer="91"/>
 <pinref part="GND10" gate="1" pin="GND"/>
-</segment>
-<segment>
-<pinref part="X3" gate="-6" pin="S"/>
-<wire x1="254" y1="15.24" x2="248.92" y2="15.24" width="0.1524" layer="91"/>
-<pinref part="GND11" gate="1" pin="GND"/>
+<pinref part="X1" gate="-5" pin="S"/>
 </segment>
 <segment>
@@
 </segment>
 <segment>
+<wire x1="254" y1="15.24" x2="248.92" y2="15.24" width="0.1524" layer="91"/>
+<label x="248.92" y="15.24" size="1.778" layer="95" rot="R180"/>
+<pinref part="JP5" gate="G$1" pin="5"/>
+</segment>
+</net>
+<net name="GPIO2" class="0">
+<segment>
+<pinref part="JP3" gate="G$1" pin="2"/>
+<wire x1="43.18" y1="38.1" x2="48.26" y2="38.1" width="0.1524" layer="91"/>
+<label x="48.26" y="38.1" size="1.778" layer="95"/>
+</segment>
+<segment>
+<wire x1="254" y1="12.7" x2="248.92" y2="12.7" width="0.1524" layer="91"/>
+<label x="248.92" y="12.7" size="1.778" layer="95" rot="R180"/>
+<pinref part="JP5" gate="G$1" pin="6"/>
+</segment>
+</net>
+<net name="GPIO3" class="0">
+<segment>
+<pinref part="JP3" gate="G$1" pin="3"/>
+<wire x1="43.18" y1="35.56" x2="48.26" y2="35.56" width="0.1524" layer="91"/>
+<label x="48.26" y="35.56" size="1.778" layer="95"/>
+</segment>
+<segment>
 <pinref part="Q1" gate="G$1" pin="G"/>
 <wire x1="187.96" y1="25.4" x2="185.42" y2="25.4" width="0.1524" layer="91"/>
 <label x="185.42" y="25.4" size="1.778" layer="95" rot="R180"/>
-</segment>
-</net>
-<net name="GPIO2" class="0">
-<segment>
-<pinref part="JP3" gate="G$1" pin="2"/>
-<wire x1="43.18" y1="38.1" x2="48.26" y2="38.1" width="0.1524" layer="91"/>
-<label x="48.26" y="38.1" size="1.778" layer="95"/>
-</segment>
-</net>
-<net name="GPIO3" class="0">
-<segment>
-<pinref part="JP3" gate="G$1" pin="3"/>
-<wire x1="43.18" y1="35.56" x2="48.26" y2="35.56" width="0.1524" layer="91"/>
-<label x="48.26" y="35.56" size="1.778" layer="95"/>
 </segment>
 </net>
@@
 </segment>
 </net>
-<net name="V_BAT" class="0">
-<segment>
-<pinref part="X2" gate="-1" pin="S"/>
-<wire x1="228.6" y1="27.94" x2="223.52" y2="27.94" width="0.1524" layer="91"/>
-<label x="223.52" y="27.94" size="1.778" layer="95" rot="R180"/>
-</segment>
-<segment>
-<pinref part="X3" gate="-1" pin="S"/>
-<wire x1="254" y1="27.94" x2="248.92" y2="27.94" width="0.1524" layer="91"/>
-<label x="248.92" y="27.94" size="1.778" layer="95" rot="R180"/>
-</segment>
-</net>
 <net name="HP0" class="0">
 <segment>
-<pinref part="X2" gate="-2" pin="S"/>
 <wire x1="228.6" y1="25.4" x2="223.52" y2="25.4" width="0.1524" layer="91"/>
 <label x="223.52" y="25.4" size="1.778" layer="95" rot="R180"/>
+<pinref part="X1" gate="-1" pin="S"/>
 </segment>
 <segment>
@@
 <net name="HP1" class="0">
 <segment>
-<pinref part="X2" gate="-3" pin="S"/>
 <wire x1="228.6" y1="22.86" x2="223.52" y2="22.86" width="0.1524" layer="91"/>
 <label x="223.52" y="22.86" size="1.778" layer="95" rot="R180"/>
+<pinref part="X1" gate="-2" pin="S"/>
 </segment>
 <segment>
@@
 <net name="HP2" class="0">
 <segment>
-<pinref part="X2" gate="-4" pin="S"/>
 <wire x1="228.6" y1="20.32" x2="223.52" y2="20.32" width="0.1524" layer="91"/>
 <label x="223.52" y="20.32" size="1.778" layer="95" rot="R180"/>
+<pinref part="X1" gate="-3" pin="S"/>
 </segment>
 <segment>
@@
 <net name="HP3" class="0">
 <segment>
-<pinref part="X2" gate="-5" pin="S"/>
 <wire x1="228.6" y1="17.78" x2="223.52" y2="17.78" width="0.1524" layer="91"/>
 <label x="223.52" y="17.78" size="1.778" layer="95" rot="R180"/>
+<pinref part="X1" gate="-4" pin="S"/>
 </segment>
 <segment>
@@
 <net name="P7" class="0">
 <segment>
-<pinref part="X3" gate="-5" pin="S"/>
 <wire x1="254" y1="17.78" x2="248.92" y2="17.78" width="0.1524" layer="91"/>
 <label x="248.92" y="17.78" size="1.778" layer="95" rot="R180"/>
+<pinref part="JP5" gate="G$1" pin="4"/>
 </segment>
 <segment>
@@
 <net name="P6" class="0">
 <segment>
-<pinref part="X3" gate="-4" pin="S"/>
 <wire x1="254" y1="20.32" x2="248.92" y2="20.32" width="0.1524" layer="91"/>
 <label x="248.92" y="20.32" size="1.778" layer="95" rot="R180"/>
+<pinref part="JP5" gate="G$1" pin="3"/>
 </segment>
 <segment>
@@
 <net name="P5" class="0">
 <segment>
-<pinref part="X3" gate="-3" pin="S"/>
 <wire x1="254" y1="22.86" x2="248.92" y2="22.86" width="0.1524" layer="91"/>
 <label x="248.92" y="22.86" size="1.778" layer="95" rot="R180"/>
+<pinref part="JP5" gate="G$1" pin="2"/>
 </segment>
 <segment>
@@
 <net name="P4" class="0">
 <segment>
-<pinref part="X3" gate="-2" pin="S"/>
 <wire x1="254" y1="25.4" x2="248.92" y2="25.4" width="0.1524" layer="91"/>
 <label x="248.92" y="25.4" size="1.778" layer="95" rot="R180"/>
+<pinref part="JP5" gate="G$1" pin="1"/>
 </segment>
 <segment>
@@
 </segment>
 </net>
+<net name="N$6" class="0">
+<segment>
+<pinref part="U$1" gate="G$1" pin="11_RF_IN"/>
+<pinref part="U$9" gate="G$1" pin="FEED"/>
+<wire x1="20.32" y1="99.06" x2="25.4" y2="99.06" width="0.1524" layer="91"/>
+</segment>
+</net>

Commit message: Board routing complete
Parts:
- added C8, C9: 100n, rcl:C-EUC0402
Connections:
- net GND: now also C8.2, C9.2
- net VCC: now also C8.1, C9.1
Changed lines of the file:
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@@
 <part name="JP5" library="SparkFun" deviceset="M06" device="SIP"/>
 <part name="U$9" library="Ava" deviceset="JTI_ANTENNA-1575AT43A40" device=""/>
+<part name="C8" library="rcl" deviceset="C-EU" device="C0402" value="100n"/>
+<part name="C9" library="rcl" deviceset="C-EU" device="C0402" value="100n"/>
 </parts>
 <sheets>
@@
 <attribute name="OC_FARNELL" x="157.48" y="88.9" size="1.778" layer="96" display="off"/>
 </instance>
-<instance part="P+6" gate="VCC" x="142.24" y="96.52"/>
+<instance part="P+6" gate="VCC" x="142.24" y="101.6"/>
 <instance part="GND7" gate="1" x="139.7" y="78.74"/>
 <instance part="U$3" gate="G$1" x="193.04" y="38.1">
@@
 <instance part="JP5" gate="G$1" x="259.08" y="20.32" rot="R180"/>
 <instance part="U$9" gate="G$1" x="12.7" y="99.06" rot="R180"/>
+<instance part="C8" gate="G$1" x="139.7" y="91.44"/>
+<instance part="C9" gate="G$1" x="238.76" y="83.82"/>
 </instances>
 <busses>
@@
 <wire x1="139.7" y1="86.36" x2="139.7" y2="81.28" width="0.1524" layer="91"/>
 <pinref part="GND7" gate="1" pin="GND"/>
+<pinref part="C8" gate="G$1" pin="2"/>
+<junction x="139.7" y="86.36"/>
 </segment>
 <segment>
@@
 <wire x1="205.74" y1="73.66" x2="203.2" y2="73.66" width="0.1524" layer="91"/>
 <junction x="203.2" y="73.66"/>
+<pinref part="C9" gate="G$1" pin="2"/>
+<wire x1="218.44" y1="66.04" x2="238.76" y2="66.04" width="0.1524" layer="91"/>
+<wire x1="238.76" y1="66.04" x2="238.76" y2="78.74" width="0.1524" layer="91"/>
 </segment>
 <segment>
@@
 <pinref part="U3" gate="G$1" pin="VDD"/>
 <wire x1="142.24" y1="91.44" x2="142.24" y2="93.98" width="0.1524" layer="91"/>
+<wire x1="142.24" y1="93.98" x2="142.24" y2="99.06" width="0.1524" layer="91"/>
 <wire x1="144.78" y1="91.44" x2="142.24" y2="91.44" width="0.1524" layer="91"/>
 <junction x="142.24" y="91.44"/>
+<pinref part="C8" gate="G$1" pin="1"/>
+<wire x1="139.7" y1="93.98" x2="142.24" y2="93.98" width="0.1524" layer="91"/>
+<junction x="142.24" y="93.98"/>
 </segment>
 <segment>
@@
 <pinref part="P+7" gate="VCC" pin="VCC"/>
 <wire x1="218.44" y1="101.6" x2="218.44" y2="99.06" width="0.1524" layer="91"/>
-</segment>
-</net>
+<pinref part="C9" gate="G$1" pin="1"/>
+<wire x1="238.76" y1="86.36" x2="238.76" y2="101.6" width="0.1524" layer="91"/>
+<wire x1="238.76" y1="101.6" x2="218.44" y2="101.6" width="0.1524" layer="91"/>
+<junction x="218.44" y="101.6"/>
+</segment>
+</net>

Commit message: shuffled rf stuffs
Parts:
- added C10, C11: (no value), rcl:C-EUC0603
Connections:
- new net N$7: C10.2, C11.1, U$1.11_RF_IN
- net GND: now also C11.2
- net N$6: now also C10.1; no longer U$1.11_RF_IN
Changed lines of the file:
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@@
 <part name="C8" library="rcl" deviceset="C-EU" device="C0402" value="100n"/>
 <part name="C9" library="rcl" deviceset="C-EU" device="C0402" value="100n"/>
+<part name="C10" library="rcl" deviceset="C-EU" device="C0603"/>
+<part name="C11" library="rcl" deviceset="C-EU" device="C0603"/>
 </parts>
 <sheets>
@@
 <instance part="X1" gate="-5" x="231.14" y="15.24"/>
 <instance part="JP5" gate="G$1" x="259.08" y="20.32" rot="R180"/>
-<instance part="U$9" gate="G$1" x="12.7" y="99.06" rot="R180"/>
+<instance part="U$9" gate="G$1" x="-7.62" y="99.06" rot="R180"/>
 <instance part="C8" gate="G$1" x="139.7" y="91.44"/>
 <instance part="C9" gate="G$1" x="238.76" y="83.82"/>
+<instance part="C10" gate="G$1" x="5.08" y="99.06" rot="R90"/>
+<instance part="C11" gate="G$1" x="17.78" y="101.6" rot="R180"/>
 </instances>
 <busses>
@@
 <wire x1="22.86" y1="104.14" x2="25.4" y2="104.14" width="0.1524" layer="91"/>
 <junction x="22.86" y="93.98"/>
+<pinref part="C11" gate="G$1" pin="2"/>
+<wire x1="22.86" y1="104.14" x2="22.86" y2="106.68" width="0.1524" layer="91"/>
+<wire x1="22.86" y1="106.68" x2="17.78" y2="106.68" width="0.1524" layer="91"/>
+<junction x="22.86" y="104.14"/>
 </segment>
 <segment>
@@
 <net name="N$6" class="0">
 <segment>
+<pinref part="U$9" gate="G$1" pin="FEED"/>
+<pinref part="C10" gate="G$1" pin="1"/>
+<wire x1="0" y1="99.06" x2="2.54" y2="99.06" width="0.1524" layer="91"/>
+</segment>
+</net>
+<net name="N$7" class="0">
+<segment>
+<pinref part="C10" gate="G$1" pin="2"/>
+<pinref part="C11" gate="G$1" pin="1"/>
+<wire x1="10.16" y1="99.06" x2="17.78" y2="99.06" width="0.1524" layer="91"/>
 <pinref part="U$1" gate="G$1" pin="11_RF_IN"/>
-<pinref part="U$9" gate="G$1" pin="FEED"/>
-<wire x1="20.32" y1="99.06" x2="25.4" y2="99.06" width="0.1524" layer="91"/>
-</segment>
-</net>
+<wire x1="17.78" y1="99.06" x2="25.4" y2="99.06" width="0.1524" layer="91"/>
+<junction x="17.78" y="99.06"/>
+</segment>
+</net>

Commit message: Changed buzzer routed lines
Parts:
- U$3: value KSSG74B16 -> KSSG23J12; device mattsLib:KSSG74B16 -> mattsLib:KSSG23J12
Changed lines of the file:
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@@
 <part name="P+6" library="supply1" deviceset="VCC" device=""/>
 <part name="GND7" library="supply1" deviceset="GND" device=""/>
-<part name="U$3" library="mattsLib" deviceset="KSSG74B16" device="">
+<part name="U$3" library="mattsLib" deviceset="KSSG23J12" device="">
 <attribute name="OC_FARNELL" value="2215090"/>
 </part>
