File: long-3.3v.sch (EAGLE design)
At the start: 45 parts, among them J1 CON_HEADER_1X06-SMD-RIGHT-ANG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, Q1 BSS84, U2 MCP73831, U3 MCP9808T-E/MC, X1 Micro USB, X2 CRYSTAL, X3 CRYSTALS-NOGND-IQXC-25

Commit message: Peer review complete, freeze design here!
Parts:
- added D1: POWER, SparkFun:LED0603
- added R11: 330, SparkFun:RESISTOR0402-RES
- U$5: OC_FARNELL (none) -> 2136254
Connections:
- new net N$8: D1.A, R11.1
- new net N$9: R11.2, U$1.PB2
- net GND: now also D1.C, U$3.P$1, U$3.P$16
Other:
- moved on the sheet: C14, U3
Changed lines of the file:
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@@
 <part name="Q1" library="transistor-small-signal" deviceset="BSS84" device=""/>
 <part name="P+8" library="supply1" deviceset="VCC" device=""/>
-<part name="U$5" library="mattsLib" deviceset="S25FL256" device=""/>
+<part name="U$5" library="mattsLib" deviceset="S25FL256" device="">
+<attribute name="OC_FARNELL" value="2136254"/>
+</part>
 <part name="P+3" library="supply1" deviceset="VCC" device=""/>
 <part name="GND4" library="supply1" deviceset="GND" device=""/>
@@
 <part name="C16" library="rcl" deviceset="C-EU" device="C0402"/>
 <part name="C17" library="rcl" deviceset="C-EU" device="C0402"/>
+<part name="GND8" library="supply1" deviceset="GND" device=""/>
+<part name="D1" library="SparkFun" deviceset="LED" device="0603" value="POWER"/>
+<part name="R11" library="SparkFun" deviceset="RESISTOR" device="0402-RES" value="330"/>
+<part name="GND10" library="supply1" deviceset="GND" device=""/>
 </parts>
 <sheets>
@@
 <instance part="C12" gate="G$1" x="-15.24" y="121.92"/>
 <instance part="C13" gate="G$1" x="-5.08" y="121.92"/>
-<instance part="U3" gate="A" x="294.64" y="116.84"/>
-<instance part="P+12" gate="VCC" x="276.86" y="132.08"/>
-<instance part="GND13" gate="1" x="276.86" y="96.52"/>
-<instance part="C14" gate="G$1" x="274.32" y="106.68"/>
+<instance part="U3" gate="A" x="299.72" y="116.84"/>
+<instance part="P+12" gate="VCC" x="281.94" y="132.08"/>
+<instance part="GND13" gate="1" x="281.94" y="96.52"/>
+<instance part="C14" gate="G$1" x="279.4" y="106.68"/>
 <instance part="J1" gate="J" x="134.62" y="68.58"/>
 <instance part="R7" gate="G$1" x="167.64" y="66.04" rot="R270"/>
 <instance part="Q1" gate="G$1" x="154.94" y="35.56"/>
 <instance part="P+8" gate="VCC" x="154.94" y="45.72"/>
-<instance part="U$5" gate="G$1" x="142.24" y="121.92"/>
+<instance part="U$5" gate="G$1" x="142.24" y="121.92">
+<attribute name="OC_FARNELL" x="142.24" y="121.92" size="1.778" layer="96" display="off"/>
+</instance>
 <instance part="P+3" gate="VCC" x="160.02" y="137.16"/>
 <instance part="GND4" gate="1" x="142.24" y="101.6"/>
@@
 <instance part="C16" gate="G$1" x="248.92" y="106.68" rot="R90"/>
 <instance part="C17" gate="G$1" x="246.38" y="101.6" rot="R180"/>
+<instance part="GND8" gate="1" x="198.12" y="132.08"/>
+<instance part="D1" gate="G$1" x="0" y="63.5"/>
+<instance part="R11" gate="G$1" x="0" y="73.66" rot="R90"/>
+<instance part="GND10" gate="1" x="0" y="55.88"/>
 </instances>
 <busses>
@@
 <wire x1="246.38" y1="99.06" x2="246.38" y2="96.52" width="0.1524" layer="91"/>
 <junction x="246.38" y="96.52"/>
+<pinref part="U$3" gate="G$1" pin="P$16"/>
+<wire x1="238.76" y1="137.16" x2="243.84" y2="137.16" width="0.1524" layer="91"/>
+<wire x1="243.84" y1="137.16" x2="243.84" y2="111.76" width="0.1524" layer="91"/>
+<junction x="243.84" y="111.76"/>
 </segment>
 <segment>
@@
 <pinref part="U3" gate="A" pin="EPAD"/>
 <pinref part="GND13" gate="1" pin="GND"/>
-<wire x1="279.4" y1="101.6" x2="276.86" y2="101.6" width="0.1524" layer="91"/>
-<wire x1="276.86" y1="101.6" x2="276.86" y2="99.06" width="0.1524" layer="91"/>
+<wire x1="284.48" y1="101.6" x2="281.94" y2="101.6" width="0.1524" layer="91"/>
+<wire x1="281.94" y1="101.6" x2="281.94" y2="99.06" width="0.1524" layer="91"/>
 <pinref part="U3" gate="A" pin="GND"/>
-<wire x1="279.4" y1="104.14" x2="276.86" y2="104.14" width="0.1524" layer="91"/>
-<wire x1="276.86" y1="104.14" x2="276.86" y2="101.6" width="0.1524" layer="91"/>
-<junction x="276.86" y="101.6"/>
+<wire x1="284.48" y1="104.14" x2="281.94" y2="104.14" width="0.1524" layer="91"/>
+<wire x1="281.94" y1="104.14" x2="281.94" y2="101.6" width="0.1524" layer="91"/>
+<junction x="281.94" y="101.6"/>
 <pinref part="C14" gate="G$1" pin="2"/>
-<wire x1="276.86" y1="101.6" x2="274.32" y2="101.6" width="0.1524" layer="91"/>
+<wire x1="281.94" y1="101.6" x2="279.4" y2="101.6" width="0.1524" layer="91"/>
 </segment>
 <segment>
@@
 <pinref part="R10" gate="G$1" pin="2"/>
 <wire x1="185.42" y1="43.18" x2="185.42" y2="45.72" width="0.1524" layer="91"/>
+</segment>
+<segment>
+<pinref part="GND8" gate="1" pin="GND"/>
+<pinref part="U$3" gate="G$1" pin="P$1"/>
+<wire x1="198.12" y1="134.62" x2="198.12" y2="137.16" width="0.1524" layer="91"/>
+<wire x1="198.12" y1="137.16" x2="208.28" y2="137.16" width="0.1524" layer="91"/>
+</segment>
+<segment>
+<pinref part="D1" gate="G$1" pin="C"/>
+<pinref part="GND10" gate="1" pin="GND"/>
 </segment>
 </net>
@@
 <pinref part="U3" gate="A" pin="A0"/>
 <pinref part="P+12" gate="VCC" pin="VCC"/>
-<wire x1="279.4" y1="109.22" x2="276.86" y2="109.22" width="0.1524" layer="91"/>
-<wire x1="276.86" y1="109.22" x2="276.86" y2="111.76" width="0.1524" layer="91"/>
+<wire x1="284.48" y1="109.22" x2="281.94" y2="109.22" width="0.1524" layer="91"/>
+<wire x1="281.94" y1="109.22" x2="281.94" y2="111.76" width="0.1524" layer="91"/>
 <pinref part="U3" gate="A" pin="A1"/>
-<wire x1="276.86" y1="111.76" x2="276.86" y2="114.3" width="0.1524" layer="91"/>
-<wire x1="276.86" y1="114.3" x2="276.86" y2="127" width="0.1524" layer="91"/>
-<wire x1="276.86" y1="127" x2="276.86" y2="129.54" width="0.1524" layer="91"/>
-<wire x1="279.4" y1="111.76" x2="276.86" y2="111.76" width="0.1524" layer="91"/>
-<junction x="276.86" y="111.76"/>
+<wire x1="281.94" y1="111.76" x2="281.94" y2="114.3" width="0.1524" layer="91"/>
+<wire x1="281.94" y1="114.3" x2="281.94" y2="127" width="0.1524" layer="91"/>
+<wire x1="281.94" y1="127" x2="281.94" y2="129.54" width="0.1524" layer="91"/>
+<wire x1="284.48" y1="111.76" x2="281.94" y2="111.76" width="0.1524" layer="91"/>
+<junction x="281.94" y="111.76"/>
 <pinref part="U3" gate="A" pin="A2"/>
-<wire x1="279.4" y1="114.3" x2="276.86" y2="114.3" width="0.1524" layer="91"/>
-<junction x="276.86" y="114.3"/>
+<wire x1="284.48" y1="114.3" x2="281.94" y2="114.3" width="0.1524" layer="91"/>
+<junction x="281.94" y="114.3"/>
 <pinref part="U3" gate="A" pin="VDD"/>
-<wire x1="279.4" y1="127" x2="276.86" y2="127" width="0.1524" layer="91"/>
-<junction x="276.86" y="127"/>
+<wire x1="284.48" y1="127" x2="281.94" y2="127" width="0.1524" layer="91"/>
+<junction x="281.94" y="127"/>
 <pinref part="C14" gate="G$1" pin="1"/>
-<wire x1="276.86" y1="109.22" x2="274.32" y2="109.22" width="0.1524" layer="91"/>
-<junction x="276.86" y="109.22"/>
+<wire x1="281.94" y1="109.22" x2="279.4" y2="109.22" width="0.1524" layer="91"/>
+<junction x="281.94" y="109.22"/>
 </segment>
 <segment>
@@
 <segment>
 <pinref part="U$3" gate="G$1" pin="P$12"/>
-<wire x1="238.76" y1="116.84" x2="243.84" y2="116.84" width="0.1524" layer="91"/>
-<label x="243.84" y="116.84" size="1.778" layer="95"/>
+<wire x1="238.76" y1="116.84" x2="246.38" y2="116.84" width="0.1524" layer="91"/>
+<label x="246.38" y="116.84" size="1.778" layer="95"/>
 </segment>
 <segment>
@@
 <segment>
 <pinref part="U$3" gate="G$1" pin="P$13"/>
-<wire x1="238.76" y1="121.92" x2="243.84" y2="121.92" width="0.1524" layer="91"/>
-<label x="243.84" y="121.92" size="1.778" layer="95"/>
+<wire x1="238.76" y1="121.92" x2="246.38" y2="121.92" width="0.1524" layer="91"/>
+<label x="246.38" y="121.92" size="1.778" layer="95"/>
 </segment>
 <segment>
@@
 <segment>
 <pinref part="U$3" gate="G$1" pin="P$14"/>
-<wire x1="238.76" y1="127" x2="243.84" y2="127" width="0.1524" layer="91"/>
-<label x="243.84" y="127" size="1.778" layer="95"/>
+<wire x1="238.76" y1="127" x2="246.38" y2="127" width="0.1524" layer="91"/>
+<label x="246.38" y="127" size="1.778" layer="95"/>
 </segment>
 <segment>
@@
 <segment>
 <pinref part="U$3" gate="G$1" pin="P$15"/>
-<wire x1="238.76" y1="132.08" x2="243.84" y2="132.08" width="0.1524" layer="91"/>
-<label x="243.84" y="132.08" size="1.778" layer="95"/>
+<wire x1="238.76" y1="132.08" x2="246.38" y2="132.08" width="0.1524" layer="91"/>
+<label x="246.38" y="132.08" size="1.778" layer="95"/>
 </segment>
 <segment>
@@
 <segment>
 <pinref part="U3" gate="A" pin="SCL"/>
-<wire x1="279.4" y1="119.38" x2="274.32" y2="119.38" width="0.1524" layer="91"/>
-<label x="274.32" y="119.38" size="1.778" layer="95" rot="R180"/>
+<wire x1="284.48" y1="119.38" x2="279.4" y2="119.38" width="0.1524" layer="91"/>
+<label x="279.4" y="119.38" size="1.778" layer="95" rot="R180"/>
 </segment>
 <segment>
@@
 <segment>
 <pinref part="U3" gate="A" pin="SDA"/>
-<wire x1="279.4" y1="121.92" x2="274.32" y2="121.92" width="0.1524" layer="91"/>
-<label x="274.32" y="121.92" size="1.778" layer="95" rot="R180"/>
+<wire x1="284.48" y1="121.92" x2="279.4" y2="121.92" width="0.1524" layer="91"/>
+<label x="279.4" y="121.92" size="1.778" layer="95" rot="R180"/>
 </segment>
 <segment>
@@
 </segment>
 </net>
+<net name="N$8" class="0">
+<segment>
+<wire x1="0" y1="68.58" x2="0" y2="66.04" width="0.1524" layer="91"/>
+<pinref part="D1" gate="G$1" pin="A"/>
+<pinref part="R11" gate="G$1" pin="1"/>
+</segment>
+</net>
+<net name="N$9" class="0">
+<segment>
+<pinref part="U$1" gate="G$1" pin="PB2"/>
+<pinref part="R11" gate="G$1" pin="2"/>
+<wire x1="35.56" y1="91.44" x2="0" y2="91.44" width="0.1524" layer="91"/>
+<wire x1="0" y1="91.44" x2="0" y2="78.74" width="0.1524" layer="91"/>
+</segment>
+</net>
